File: Hardware/SparkFun_Photon_Weather_Shield.sch (EAGLE design)
At the start: 44 parts, among them U1 3.3V MIC5219, U2 HTU21D, U3 MPL3115A2LGA8

Commit message: Updating Example Sketches
Updating Example Sketches
Other:
- note added: "Max Voltage Input on Photon VIN: 5.5-6VDC"
Changed lines of the file:
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@@
 <text x="165.862" y="11.176" size="2.54" layer="94">Joel Bartlett</text>
 <text x="236.22" y="7.62" size="2.54" layer="94">V10</text>
+<text x="144.78" y="172.72" size="1.778" layer="97">Max Voltage Input on Photon VIN: 5.5-6VDC</text>
 </plain>
 <instances>

Commit message: Initial Commit to V11
Parts:
- U2: value HTU21D -> SI7021; device SparkFun-Sensors:HTU21DSMD -> SparkFun-Sensors:SI7021
Connections:
- net GND: now also U2.GND; no longer U2.GND@2, U2.GND@7
Other:
- note added: "V11"
- note removed: "V10"
Changed lines of the file:
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@@
 <part name="P+7" library="SparkFun" deviceset="VCC" device="" value="3.3V"/>
 <part name="GND12" library="SparkFun" deviceset="GND" device=""/>
-<part name="U2" library="SparkFun-Sensors" deviceset="HTU21D" device="SMD" value="HTU21D"/>
 <part name="P+4" library="SparkFun" deviceset="VCC" device="" value="3.3V"/>
 <part name="P+3" library="SparkFun" deviceset="VCC" device="" value="3.3V"/>
@@
 <part name="LOGO2" library="SparkFun-Aesthetics" deviceset="SFE_LOGO_NAME" device=".1_INCH"/>
 <part name="FRAME1" library="SparkFun-Aesthetics" deviceset="FRAME-LETTER" device=""/>
+<part name="U2" library="SparkFun-Sensors" deviceset="SI7021" device=""/>
 </parts>
 <sheets>
@@
 <text x="60.452" y="122.428" size="2.032" layer="102">Serial 1 Port (optional)</text>
 <text x="165.862" y="11.176" size="2.54" layer="94">Joel Bartlett</text>
-<text x="236.22" y="7.62" size="2.54" layer="94">V10</text>
+<text x="236.22" y="7.62" size="2.54" layer="94">V11</text>
 <text x="144.78" y="172.72" size="1.778" layer="97">Max Voltage Input on Photon VIN: 5.5-6VDC</text>
 </plain>
@@
 <instance part="P+7" gate="1" x="5.08" y="116.84"/>
 <instance part="GND12" gate="1" x="15.24" y="101.6"/>
-<instance part="U2" gate="U$1" x="27.94" y="109.22"/>
 <instance part="P+4" gate="1" x="35.56" y="76.2"/>
 <instance part="P+3" gate="1" x="5.08" y="71.12"/>
@@
 <attribute name="DRAWING_NAME" x="162.814" y="17.78" size="2.7432" layer="94" font="vector"/>
 </instance>
+<instance part="U2" gate="G$1" x="27.94" y="109.22"/>
 </instances>
 <busses>
@@
 </segment>
 <segment>
-<wire x1="17.78" y1="106.68" x2="15.24" y2="106.68" width="0.1524" layer="91"/>
-<wire x1="15.24" y1="106.68" x2="15.24" y2="104.14" width="0.1524" layer="91"/>
 <pinref part="GND12" gate="1" pin="GND"/>
-<pinref part="U2" gate="U$1" pin="GND@7"/>
-<pinref part="U2" gate="U$1" pin="GND@2"/>
 <wire x1="17.78" y1="109.22" x2="15.24" y2="109.22" width="0.1524" layer="91"/>
-<wire x1="15.24" y1="109.22" x2="15.24" y2="106.68" width="0.1524" layer="91"/>
-<junction x="15.24" y="106.68"/>
+<wire x1="15.24" y1="109.22" x2="15.24" y2="104.14" width="0.1524" layer="91"/>
+<pinref part="U2" gate="G$1" pin="GND"/>
 </segment>
 <segment>
@@
 <segment>
 <wire x1="17.78" y1="111.76" x2="15.24" y2="111.76" width="0.1524" layer="91"/>
-<pinref part="U2" gate="U$1" pin="VDD"/>
 <pinref part="P+13" gate="1" pin="VCC"/>
 <wire x1="15.24" y1="114.3" x2="15.24" y2="111.76" width="0.1524" layer="91"/>
+<pinref part="U2" gate="G$1" pin="VDD"/>
 </segment>
 <segment>
@@
 </segment>
 <segment>
-<pinref part="U2" gate="U$1" pin="SCK"/>
 <label x="40.64" y="109.22" size="1.27" layer="95" xref="yes"/>
 <wire x1="38.1" y1="109.22" x2="40.64" y2="109.22" width="0.1524" layer="91"/>
+<pinref part="U2" gate="G$1" pin="SCK"/>
 </segment>
 <segment>
@@
 </segment>
 <segment>
-<pinref part="U2" gate="U$1" pin="DATA"/>
 <label x="40.64" y="111.76" size="1.27" layer="95" xref="yes"/>
 <wire x1="38.1" y1="111.76" x2="40.64" y2="111.76" width="0.1524" layer="91"/>
-</segment>
-<segment>
+<pinref part="U2" gate="G$1" pin="DATA"/>
+</segment>
+<segment>
