File: Hardware/SparkFun_Photon_Weather_Shield.sch (EAGLE design)
At the start: 44 parts, among them U1 3.3V MIC5219, U2 HTU21D, U3 MPL3115A2LGA8

Commit message: Update w/ Correct Voltage Regulator Name
The schematic was updated incorrectly with the voltage regulator name and specifications. Instead of the MIC5219, it is populated with the **MIC5205**.

While the recommended operating voltage from the [datasheet](http://ww1.microchip.com/downloads/en/DeviceDoc/20005785A.pdf) is up to +16V, the actual stable voltage in real world conditions is actually about ~11.5V. This has been been tested and verified by @sfemark .
Parts:
- U1: value 3.3V MIC5219 -> 3.3V MIC5205
Other:
- note added: "Max Current Output: 150mA"
- note added: "Max Voltage Input: ~11.5VDC"
- note removed: "Max Current Output: 500mA"
- note removed: "Max Voltage Input: 12VDC"
Changed lines of the file:
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@@
 <?xml version="1.0" encoding="utf-8"?>
 <!DOCTYPE eagle SYSTEM "eagle.dtd">
-<eagle version="7.2.0">
+<eagle version="7.6.0">
 <drawing>
 <settings>
@@
 <part name="GND25" library="SparkFun" deviceset="GND" device=""/>
 <part name="GND26" library="SparkFun" deviceset="GND" device=""/>
-<part name="U1" library="SparkFun-PowerIC" deviceset="MIC5205" device="3.3V" value="3.3V MIC5219"/>
+<part name="U1" library="SparkFun-PowerIC" deviceset="MIC5205" device="3.3V" value="3.3V MIC5205"/>
 <part name="GND30" library="SparkFun" deviceset="GND" device=""/>
 <part name="C1" library="SparkFun-Capacitors" deviceset="1.0UF-16V-10%(0603)" device="" value="1.0uF"/>
@@
 <sheet>
 <plain>
-<text x="27.94" y="147.32" size="1.778" layer="97">Max Voltage Input: 12VDC</text>
-<text x="27.94" y="142.24" size="1.778" layer="97">Max Current Output: 500mA</text>
+<text x="27.94" y="147.32" size="1.778" layer="97">Max Voltage Input: ~11.5VDC</text>
+<text x="27.94" y="142.24" size="1.778" layer="97">Max Current Output: 150mA</text>
 <text x="40.64" y="53.34" size="1.778" layer="97">Read Address:</text>
 <text x="40.64" y="50.8" size="1.778" layer="97">Write Address:</text>
