File: Hardware/SparkFun_Photon_Weather_Shield_V11.brd (EAGLE design)
At the start: 71.1 x 35.6 mm, 46 parts, among them U1 3.3V MIC5219, U2 SI7021, U3 MPL3115A2LGA8

Commit message: Preliminary Checklist review
Parts:
- R4, R5: value 10K -> 4.7K
- renumbered R2 to R5, R3 to R4
Changed lines of the file:
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@@
 <?xml version="1.0" encoding="utf-8"?>
 <!DOCTYPE eagle SYSTEM "eagle.dtd">
-<eagle version="7.2.0">
+<eagle version="7.6.0">
 <drawing>
 <settings>
@@
 <layer number="47" name="Measures" color="7" fill="1" visible="no" active="yes"/>
 <layer number="48" name="Document" color="7" fill="1" visible="no" active="yes"/>
-<layer number="49" name="Reference" color="7" fill="1" visible="no" active="yes"/>
+<layer number="49" name="Reference" color="7" fill="1" visible="yes" active="yes"/>
 <layer number="50" name="dxf" color="7" fill="1" visible="no" active="no"/>
 <layer number="51" name="tDocu" color="6" fill="1" visible="yes" active="yes"/>
@@
 <layer number="112" name="tSilk" color="7" fill="1" visible="no" active="yes"/>
 <layer number="113" name="IDFDebug" color="4" fill="1" visible="no" active="yes"/>
+<layer number="114" name="Badge_Outline" color="7" fill="1" visible="no" active="yes"/>
+<layer number="115" name="ReferenceISLANDS" color="7" fill="1" visible="no" active="yes"/>
 <layer number="116" name="Patch_BOT" color="9" fill="4" visible="no" active="yes"/>
 <layer number="118" name="Rect_Pads" color="7" fill="1" visible="no" active="yes"/>
@@
 <attribute name="PROD_ID" value="RES-07857" x="66.04" y="2.54" size="1.778" layer="27" font="vector" ratio="15" rot="R90" display="off"/>
 </element>
-<element name="JP1" library="SparkFun-Connectors" package="1X04" value="I2C Port" x="69.85" y="5.08" rot="R90"/>
+<element name="JP1" library="SparkFun-Connectors" package="1X04" value="I2C Port" x="69.85" y="5.08" rot="R90">
+<attribute name="PROD_ID" value="CONN-09696" x="69.85" y="5.08" size="1.778" layer="27" rot="R90" display="off"/>
+</element>
 <element name="SJ1" library="SparkFun-Passives" package="PAD-JUMPER-3-3OF3_NC_BY_TRACE_YES_SILK_FULL_BOX" value="" x="66.675" y="15.875" rot="R180"/>
-<element name="R2" library="SparkFun-Resistors" package="0603-RES" value="10K" x="69.215" y="15.875" rot="R90">
-<attribute name="PROD_ID" value="RES-00824" x="69.215" y="15.875" size="1.778" layer="27" font="vector" ratio="15" rot="R90" display="off"/>
-</element>
-<element name="R3" library="SparkFun-Resistors" package="0603-RES" value="10K" x="64.135" y="15.875" rot="R90">
-<attribute name="PROD_ID" value="RES-00824" x="64.135" y="15.875" size="1.778" layer="27" font="vector" ratio="15" rot="R90" display="off"/>
-</element>
 <element name="JP5-DNP" library="SparkFun-Connectors" package="POWER_JACK_SMD" value="5.5x2.1mm Barrel" x="35.56" y="33.655" rot="MR270">
 <attribute name="PROD_ID" value="CONN-08106" x="35.56" y="33.655" size="1.778" layer="28" font="vector" ratio="15" rot="MR270" display="off"/>
@@
 <element name="FID2" library="SparkFun-Aesthetics" package="FIDUCIAL-1X2" value="FIDUCIAL1X2" x="15.875" y="29.845"/>
 <element name="SJ3" library="SparkFun-Passives" package="PAD-JUMPER-2-NC_BY_TRACE_YES_SILK" value="" x="35.56" y="16.51" rot="MR180"/>
-<element name="JP4" library="SparkFun-Connectors" package="1X04" value="Serial1 Port" x="1.27" y="5.08" rot="R90"/>
+<element name="JP4" library="SparkFun-Connectors" package="1X04" value="Serial1 Port" x="1.27" y="5.08" rot="R90">
+<attribute name="PROD_ID" value="CONN-09696" x="1.27" y="5.08" size="1.778" layer="27" rot="R90" display="off"/>
+</element>
 <element name="U$3" library="SparkFun-Aesthetics" package="SFE_LOGO_FLAME_.1" value="" x="62.992" y="9.652"/>
 <element name="JP9" library="template_temp" package="SPARK_PHOTON_TEMPLATE_WIDE_LOCKING" value="PHOTON_TEMPLATE_WIDE_LOCKING" x="25.4" y="0"/>
@@
 <element name="U2" library="SparkFun-Sensors" package="SI7021" value="SI7021" x="8.255" y="12.7" rot="R90">
 <attribute name="PROD_ID" value="IC-13093" x="8.255" y="12.7" size="1.778" layer="27" rot="R90" display="off"/>
+</element>
+<element name="R4" library="SparkFun-Resistors" package="0603-RES" value="4.7K" x="64.135" y="15.875" rot="R90">
+<attribute name="PROD_ID" value="RES-07857" x="64.135" y="15.875" size="1.778" layer="27" font="vector" ratio="15" rot="R90" display="off"/>
+</element>
+<element name="R5" library="SparkFun-Resistors" package="0603-RES" value="4.7K" x="69.215" y="15.875" rot="R90">
+<attribute name="PROD_ID" value="RES-07857" x="69.215" y="15.875" size="1.778" layer="27" font="vector" ratio="15" rot="R90" display="off"/>
 </element>
 </elements>
@@
 <contactref element="U3" pad="8"/>
 <contactref element="JP1" pad="1"/>
-<contactref element="R3" pad="1"/>
 <wire x1="11.835" y1="11.2" x2="12.065" y2="11.43" width="0.254" layer="1"/>
 <wire x1="12.065" y1="11.43" x2="12.065" y2="13.335" width="0.254" layer="1"/>
@@
 <wire x1="64.135" y1="10.795" x2="53.975" y2="10.795" width="0.254" layer="1"/>
 <wire x1="64.135" y1="8.255" x2="64.135" y2="10.795" width="0.254" layer="1"/>
-<wire x1="64.135" y1="10.795" x2="64.135" y2="15.025" width="0.254" layer="1"/>
 <contactref element="JP9" pad="14"/>
 <contactref element="JP9" pad="D1"/>
@@
 <contactref element="U2" pad="SCK"/>
 <wire x1="11.835" y1="11.2" x2="9.255" y2="11.2" width="0.254" layer="1"/>
+<contactref element="R4" pad="1"/>
+<wire x1="64.135" y1="15.025" x2="64.135" y2="10.795" width="0.254" layer="1"/>
 </signal>
 <signal name="SDA">
 <contactref element="U3" pad="7"/>
 <contactref element="JP1" pad="2"/>
-<contactref element="R2" pad="1"/>
 <wire x1="11.66" y1="14.2" x2="12.7" y2="15.24" width="0.254" layer="1"/>
 <wire x1="14.605" y1="13.91" x2="14.615" y2="13.9" width="0.254" layer="1"/>
@@
 <wire x1="52.07" y1="5.715" x2="66.675" y2="5.715" width="0.254" layer="1"/>
 <wire x1="69.85" y1="7.62" x2="67.8688" y2="7.62" width="0.254" layer="1"/>
-<wire x1="69.215" y1="15.025" x2="69.215" y2="14.4272" width="0.254" layer="1"/>
 <wire x1="69.215" y1="14.4272" x2="69.0626" y2="14.2748" width="0.254" layer="1"/>
 <wire x1="69.0626" y1="14.2748" x2="68.5546" y2="14.2748" width="0.254" layer="1"/>
@@
 <contactref element="U2" pad="DATA"/>
 <wire x1="11.66" y1="14.2" x2="9.255" y2="14.2" width="0.254" layer="1"/>
+<contactref element="R5" pad="1"/>
+<wire x1="69.215" y1="14.4272" x2="69.215" y2="15.025" width="0.254" layer="1"/>
 </signal>
 <signal name="INT-PRESSURE">
@@
 <signal name="N$3">
 <contactref element="SJ1" pad="3"/>
-<contactref element="R3" pad="2"/>
-<wire x1="64.135" y1="16.725" x2="64.7074" y2="16.725" width="0.254" layer="1"/>
 <wire x1="64.7074" y1="16.725" x2="65.024" y2="16.4084" width="0.254" layer="1"/>
 <wire x1="65.024" y1="16.4084" x2="65.024" y2="16.1544" width="0.254" layer="1"/>
@@
 <wire x1="65.278" y1="15.9004" x2="65.8368" y2="15.9004" width="0.254" layer="1"/>
 <wire x1="65.8368" y1="15.9004" x2="65.8622" y2="15.875" width="0.254" layer="1"/>
+<contactref element="R4" pad="2"/>
+<wire x1="64.7074" y1="16.725" x2="64.135" y2="16.725" width="0.254" layer="1"/>
 </signal>
 <signal name="N$6">
-<contactref element="R2" pad="2"/>
 <contactref element="SJ1" pad="1"/>
-<wire x1="69.215" y1="16.725" x2="68.5156" y2="16.725" width="0.254" layer="1"/>
 <wire x1="68.5156" y1="16.725" x2="68.199" y2="16.4084" width="0.254" layer="1"/>
 <wire x1="68.199" y1="16.4084" x2="68.199" y2="16.0274" width="0.254" layer="1"/>
@@
 <wire x1="68.072" y1="15.9004" x2="67.5132" y2="15.9004" width="0.254" layer="1"/>
 <wire x1="67.5132" y1="15.9004" x2="67.4878" y2="15.875" width="0.254" layer="1"/>
+<contactref element="R5" pad="2"/>
+<wire x1="68.5156" y1="16.725" x2="69.215" y2="16.725" width="0.254" layer="1"/>
 </signal>
 <signal name="SOIL_MOIST1">

Commit message: Final Changes before ENG Checklist
Many minor changes: text, font, paste under Si7021 footprint. correct
layers for info.
Parts:
- renumbered JP1 to JP1-DNP, JP2 to JP2-DNP, JP3 to JP3-DNP, JP4 to JP4-DNP
Routing:
- net SCL: track 72.6 -> 75.6 mm
- net 3.3V: track 153.7 -> 152.5 mm
- net SDA: track 74.1 -> 75.1 mm

Commit message: Updates for ENG Checklist
Connections:
- removed net INT-PRESSURE: U3.6
