File: Hardware/SparkFun_Photon_Weather_Shield_V11.brd (EAGLE design)
At the start: 71.1 x 35.6 mm, 46 parts, among them U1 3.3V MIC5219, U2 SI7021, U3 MPL3115A2LGA8

Commit message: Update w/ Correct Voltage Regulator Name
The schematic was updated incorrectly with the voltage regulator name and specifications. Instead of the MIC5219, it is populated with the **MIC5205**.

While the recommended operating voltage from the [datasheet](http://ww1.microchip.com/downloads/en/DeviceDoc/20005785A.pdf) is up to +16V, the actual stable voltage in real world conditions is actually about ~11.5V. This has been been tested and verified by @sfemark .
Parts:
- U1: value 3.3V MIC5219 -> 3.3V MIC5205
