File: Hardware/SparkFun_Photon_Weather_Shield_V11.sch (EAGLE design)
At the start: 44 parts, among them U1 3.3V MIC5219, U2 SI7021, U3 MPL3115A2LGA8

Commit message: Preliminary Checklist review
Parts:
- removed R2, R3: 10K, SparkFun-Resistors:10KOHM-1/10W-1%(0603)0603
- added R4, R5: 4.7K, SparkFun-Resistors:4.7KOHM-1/10W-1%(0603)
Connections:
- net N$3: now also R4.2; no longer R3.2
- net N$6: now also R5.2; no longer R2.2
- net SCL: now also R4.1; no longer R3.1
- net SDA: now also R5.1; no longer R2.1
Other:
- moved on the sheet: SJ2

Commit message: Final Changes before ENG Checklist
Many minor changes: text, font, paste under Si7021 footprint. correct
layers for info.
Parts:
- renumbered JP1 to JP1-DNP, JP2 to JP2-DNP, JP3 to JP3-DNP, JP4 to JP4-DNP
Other:
- note added: "7-bit I2C Address: 0x40"
- note added: "7-bit I2C Address: 0x60"
- note added: "I2C Pull-up Solder Jumper"
- note added: "I2C Read: 0x81"
- note added: "I2C Read: 0xC1"
- note added: "I2C Write: 0x80"
- note added: "I2C Write: 0xC0"
- note added: "Power Select Solder Jumper"
- note removed: "0x60"
- note removed: "0xC0"
- note removed: "0xC1"
- note removed: "7-bit I2C Address is 0x40"
- note removed: "7-bit I2C Address:"
- note removed: "I2C read is 0x81"
- note removed: "I2C write is 0x80"
- note removed: "Read Address:"
- note removed: "Write Address:"

Commit message: Updates for ENG Checklist
Connections:
- removed net INT-PRESSURE: U3.INT1
Changed lines of the file:
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@@
-</segment>
-</net>
-<net name="INT-PRESSURE" class="0">
-<segment>
-<wire x1="63.5" y1="68.58" x2="66.04" y2="68.58" width="0.1524" layer="91"/>
-<pinref part="U3" gate="G$1" pin="INT1"/>
-<label x="66.04" y="68.58" size="1.27" layer="95" font="vector" xref="yes"/>
 </segment>
 </net>
